File: PoppingUnit-PCB/PoppingUnit.brd (EAGLE design)
At the start: 95 x 63 mm, 81 parts, among them IC2 7805DT, J2 POWER_JACKPTH, Q1 16MHz 10ppm, U1 ARDUINO_LEONARDO-REV3B_SMARTP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, U2 SN75176ASOIC, X1 USBPTH

Commit message: Update schematic with production component values
Parts:
- C11: value .3uF -> DNP
- C13: value .3uF -> 470nF
- C14: value 100nF -> DNP
- R18, R8: value 1k -> 330
Changed lines of the file:
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@@
 <element name="R1" library="adafruit" package="R0603" value="180 DNP" x="21" y="12.25" smashed="yes" rot="R270"/>
 <element name="R2" library="adafruit" package="R0603" value="10k" x="27.75" y="8.5" smashed="yes" rot="R180"/>
-<element name="R8" library="adafruit" package="R0603" value="1k" x="15.5" y="41.25" smashed="yes"/>
+<element name="R8" library="adafruit" package="R0603" value="330" x="15.5" y="41.25" smashed="yes"/>
 <element name="C7" library="adafruit" package="C0603K" value="100nF" x="23.75" y="8.5" smashed="yes"/>
 <element name="U$2" library="sonos_library" package="2X3HEADER" value="2X3HEADER" x="19.75" y="57.75" smashed="yes" rot="R270"/>
@@
 <element name="U$9" library="blinkinlabs" package="TO252" value="N_MOSFET" x="36" y="51" smashed="yes"/>
 <element name="C8" library="adafruit" package="C0603K" value="1uF" x="23" y="53.5" smashed="yes" rot="R90"/>
-<element name="C11" library="adafruit" package="C0603K" value=".3uF" x="37" y="41.5" smashed="yes" rot="R90"/>
+<element name="C11" library="adafruit" package="C0603K" value="DNP" x="37" y="41.5" smashed="yes" rot="R90"/>
 <element name="C12" library="adafruit" package="C0603K" value="100nF" x="28.5" y="36.5" smashed="yes" rot="R180"/>
-<element name="C13" library="adafruit" package="C0603K" value=".3uF" x="35.5" y="41.5" smashed="yes" rot="R90"/>
-<element name="C14" library="adafruit" package="C0603K" value="100nF" x="28.5" y="38" smashed="yes" rot="R180"/>
+<element name="C13" library="adafruit" package="C0603K" value="470nF" x="35.5" y="41.5" smashed="yes" rot="R90"/>
+<element name="C14" library="adafruit" package="C0603K" value="DNP" x="28.5" y="38" smashed="yes" rot="R180"/>
 <element name="LED1" library="SparkFun" package="LED5MM" value="" x="18" y="37.75" smashed="yes" rot="R270">
 <attribute name="VALUE" x="16.1966" y="34.5496" size="1.27" layer="27" ratio="10" rot="R270"/>
@@
 <attribute name="VALUE" x="5.623" y="4.84" size="1.778" layer="27"/>
 </element>
-<element name="R18" library="adafruit" package="R0603" value="1k" x="15" y="39" smashed="yes" rot="R180"/>
+<element name="R18" library="adafruit" package="R0603" value="330" x="15" y="39" smashed="yes" rot="R180"/>
 <element name="LED2" library="SparkFun" package="LED5MM" value="" x="18" y="28" smashed="yes" rot="R270">
 <attribute name="VALUE" x="16.1966" y="24.7996" size="1.27" layer="27" ratio="10" rot="R270"/>
