File: PoppingUnit-PCB/PoppingUnit.sch (EAGLE design)
At the start: 77 parts, among them IC2 7805DT, J1 RS485, J2 POWER_JACKPTH, Q1 16MHz 10ppm, U1 ARDUINO_LEONARDO-REV3B_SMARTP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, U2 SN75176ASOIC, X1 USBPTH

Commit message: Update popping unit to RevB (should be good to go!)
Parts:
- removed J1: RS485, con-amp:520426-4
- added J3: (no value), con-amp:555153-1
- added LED2: (no value), SparkFun:LED5MM
- added R18: 1k, adafruit:R-US_R0603
Connections:
- net SIG0 renamed OUT_5
- net SIG1 renamed OUT_6
- net SIG10 renamed OUT_15
- net SIG11 renamed OUT_16
- net SIG12 renamed OUT_4
- net SIG13 renamed OUT_3
- net SIG14 renamed OUT_2
- net SIG2 renamed OUT_7
- net SIG3 renamed OUT_8
- net SIG4 renamed OUT_12
- net SIG5 renamed OUT_11
- net SIG6 renamed OUT_10
- net SIG7 renamed OUT_9
- net SIG8 renamed OUT_13
- net SIG9 renamed OUT_14
- removed net SIG15: R22.2, U$18.G, U1.(#HWB)PE2
- new net OUT_1: R22.2, U$18.G, U1.(TXD1/INT3)PD3
- new net STATUS_1: R18.2, U1.(SDA/INT1)PD1
- net GND: now also J3.7, J3.8, LED2.C; no longer J1.7, J1.8
- net N$12: now also LED2.A, R18.1; no longer U1.(TXD1/INT3)PD3
- net RS485A: now also J3.1; no longer J1.1
- net RS485B: now also J3.2; no longer J1.2
- net VIN: now also J3.4, J3.5; no longer J1.4, J1.5
Changed lines of the file:
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@@
 <part name="GND12" library="supply1" deviceset="GND" device=""/>
 <part name="C7" library="adafruit" deviceset="C-US" device="C0603K" value="100nF"/>
-<part name="J1" library="con-amp" deviceset="520426-4" device="" value="RS485"/>
 <part name="U$2" library="sonos_library" deviceset="2X3HEADER" device=""/>
 <part name="GND10" library="supply1" deviceset="GND" device=""/>
@@
 <part name="SUPPLY26" library="SparkFun-Aesthetics" deviceset="VIN" device=""/>
 <part name="SUPPLY27" library="SparkFun-Aesthetics" deviceset="2.8V" device=""/>
+<part name="J3" library="con-amp" deviceset="555153-1" device=""/>
+<part name="R18" library="adafruit" deviceset="R-US_" device="R0603" value="1k"/>
+<part name="GND29" library="supply1" deviceset="GND" device=""/>
+<part name="LED2" library="SparkFun" deviceset="LED" device="5MM"/>
 </parts>
 <sheets>
@@
 <attribute name="NAME" x="49.784" y="-78.359" size="1.778" layer="95"/>
 <attribute name="VALUE" x="47.244" y="-80.899" size="1.778" layer="96"/>
-</instance>
-<instance part="J1" gate="G$1" x="30.48" y="-99.06" smashed="yes" rot="MR270">
-<attribute name="NAME" x="25.4" y="-101.6" size="1.778" layer="95" rot="MR180"/>
-<attribute name="VALUE" x="43.688" y="-93.98" size="1.778" layer="96" rot="MR270"/>
 </instance>
 <instance part="U$2" gate="G$1" x="129.54" y="53.34"/>
@@
 </instance>
 <instance part="GND2" gate="1" x="15.24" y="-104.14"/>
-<instance part="GND8" gate="1" x="45.72" y="-96.52"/>
+<instance part="GND8" gate="1" x="50.8" y="-93.98"/>
 <instance part="U$10" gate="G$1" x="273.05" y="-35.56"/>
 <instance part="GND20" gate="1" x="279.4" y="-46.99"/>
@@
 <instance part="SUPPLY26" gate="G$1" x="127" y="-66.04"/>
 <instance part="SUPPLY27" gate="G$1" x="162.56" y="-66.04"/>
+<instance part="J3" gate="G$1" x="33.02" y="-96.52" rot="MR270"/>
+<instance part="R18" gate="G$1" x="167.64" y="53.34" rot="R90"/>
+<instance part="GND29" gate="1" x="167.64" y="33.02"/>
+<instance part="LED2" gate="G$1" x="167.64" y="43.18"/>
 </instances>
 <busses>
@@
 <wire x1="139.7" y1="-20.32" x2="139.7" y2="-22.86" width="0.1524" layer="91"/>
 <junction x="139.7" y="-22.86"/>
+<junction x="165.1" y="-22.86"/>
 </segment>
 <segment>
@@
 </segment>
 <segment>
-<pinref part="J1" gate="G$1" pin="8"/>
 <wire x1="40.64" y1="-93.98" x2="38.1" y2="-93.98" width="0.1524" layer="91"/>
 <junction x="38.1" y="-93.98"/>
-<pinref part="J1" gate="G$1" pin="7"/>
 <wire x1="38.1" y1="-93.98" x2="38.1" y2="-91.44" width="0.1524" layer="91"/>
 <wire x1="38.1" y1="-91.44" x2="45.72" y2="-91.44" width="0.1524" layer="91"/>
 <pinref part="GND8" gate="1" pin="GND"/>
-<wire x1="45.72" y1="-91.44" x2="45.72" y2="-93.98" width="0.1524" layer="91"/>
+<wire x1="45.72" y1="-91.44" x2="50.8" y2="-91.44" width="0.1524" layer="91"/>
 <pinref part="C7" gate="G$1" pin="2"/>
 <wire x1="45.72" y1="-83.82" x2="45.72" y2="-91.44" width="0.1524" layer="91"/>
 <junction x="45.72" y="-91.44"/>
+<pinref part="J3" gate="G$1" pin="7"/>
+<pinref part="J3" gate="G$1" pin="8"/>
 </segment>
 <segment>
@@
 <wire x1="144.78" y1="-76.2" x2="144.78" y2="-78.74" width="0.1524" layer="91"/>
 </segment>
+<segment>
+<wire x1="167.64" y1="38.1" x2="167.64" y2="35.56" width="0.1524" layer="91"/>
+<pinref part="GND29" gate="1" pin="GND"/>
+<pinref part="LED2" gate="G$1" pin="C"/>
+</segment>
 </net>
 <net name="RX" class="0">
@@
 <pinref part="R1" gate="G$1" pin="2"/>
 <pinref part="U2" gate="G$1" pin="B"/>
-<pinref part="J1" gate="G$1" pin="2"/>
+<pinref part="J3" gate="G$1" pin="2"/>
 </segment>
 </net>
@@
 <pinref part="U2" gate="G$1" pin="A"/>
 <pinref part="R1" gate="G$1" pin="1"/>
-<pinref part="J1" gate="G$1" pin="1"/>
 <wire x1="22.86" y1="-88.9" x2="22.86" y2="-93.98" width="0.1524" layer="91"/>
 <junction x="20.32" y="-88.9"/>
+<pinref part="J3" gate="G$1" pin="1"/>
 </segment>
 </net>
@@
 </segment>
 </net>
-<net name="N$12" class="0">
-<segment>
-<pinref part="U1" gate="G$1" pin="(TXD1/INT3)PD3"/>
-<wire x1="73.66" y1="7.62" x2="76.2" y2="7.62" width="0.1524" layer="91"/>
-</segment>
-</net>
 <net name="RXLED" class="0">
 <segment>
@@
 </segment>
 </net>
-<net name="SIG0" class="0">
+<net name="OUT_5" class="0">
 <segment>
 <label x="255.27" y="63.5" size="1.778" layer="95" rot="R180" xref="yes"/>
@@
 </segment>
 </net>
-<net name="SIG1" class="0">
+<net name="OUT_6" class="0">
 <segment>
 <label x="255.27" y="36.83" size="1.778" layer="95" rot="R180" xref="yes"/>
@@
 </segment>
 </net>
-<net name="SIG2" class="0">
+<net name="OUT_7" class="0">
 <segment>
 <label x="255.27" y="10.16" size="1.778" layer="95" rot="R180" xref="yes"/>
@@
 </segment>
 </net>
-<net name="SIG3" class="0">
+<net name="OUT_8" class="0">
 <segment>
 <label x="255.27" y="-13.97" size="1.778" layer="95" rot="R180" xref="yes"/>
@@
 </segment>
 </net>
-<net name="SIG4" class="0">
+<net name="OUT_12" class="0">
 <segment>
 <label x="255.27" y="-38.1" size="1.778" layer="95" rot="R180" xref="yes"/>
@@
 </segment>
 </net>
-<net name="SIG5" class="0">
+<net name="OUT_11" class="0">
 <segment>
 <label x="255.27" y="-64.77" size="1.778" layer="95" rot="R180" xref="yes"/>
@@
 </segment>
 </net>
-<net name="SIG6" class="0">
+<net name="OUT_10" class="0">
 <segment>
 <label x="255.27" y="-91.44" size="1.778" layer="95" rot="R180" xref="yes"/>
@@
 </segment>
 </net>
-<net name="SIG7" class="0">
+<net name="OUT_9" class="0">
 <segment>
 <label x="255.27" y="-115.57" size="1.778" layer="95" rot="R180" xref="yes"/>
@@
 </segment>
 </net>
-<net name="SIG8" class="0">
+<net name="OUT_13" class="0">
 <segment>
 <label x="311.15" y="63.5" size="1.778" layer="95" rot="R180" xref="yes"/>
@@
 </segment>
 </net>
-<net name="SIG9" class="0">
+<net name="OUT_14" class="0">
 <segment>
 <label x="311.15" y="36.83" size="1.778" layer="95" rot="R180" xref="yes"/>
@@
 </segment>
 </net>
-<net name="SIG10" class="0">
+<net name="OUT_15" class="0">
 <segment>
 <label x="311.15" y="10.16" size="1.778" layer="95" rot="R180" xref="yes"/>
@@
 </segment>
 </net>
-<net name="SIG11" class="0">
+<net name="OUT_16" class="0">
 <segment>
 <label x="311.15" y="-13.97" size="1.778" layer="95" rot="R180" xref="yes"/>
@@
 </segment>
 </net>
-<net name="SIG12" class="0">
+<net name="OUT_4" class="0">
 <segment>
 <label x="311.15" y="-38.1" size="1.778" layer="95" rot="R180" xref="yes"/>
@@
 </segment>
 </net>
-<net name="SIG13" class="0">
+<net name="OUT_3" class="0">
 <segment>
 <label x="311.15" y="-64.77" size="1.778" layer="95" rot="R180" xref="yes"/>
@@
 </segment>
 </net>
-<net name="SIG14" class="0">
+<net name="OUT_2" class="0">
 <segment>
 <label x="311.15" y="-91.44" size="1.778" layer="95" rot="R180" xref="yes"/>
@@
 </segment>
 </net>
-<net name="SIG15" class="0">
+<net name="OUT_1" class="0">
 <segment>
 <label x="311.15" y="-115.57" size="1.778" layer="95" rot="R180" xref="yes"/>
@@
 </segment>
 <segment>
-<pinref part="U1" gate="G$1" pin="(#HWB)PE2"/>
-<wire x1="73.66" y1="22.86" x2="76.2" y2="22.86" width="0.1524" layer="91"/>
-<label x="76.2" y="22.86" size="1.778" layer="95" xref="yes"/>
+<pinref part="U1" gate="G$1" pin="(TXD1/INT3)PD3"/>
+<wire x1="73.66" y1="7.62" x2="76.2" y2="7.62" width="0.1524" layer="91"/>
+<label x="76.2" y="7.62" size="1.778" layer="95" xref="yes"/>
 </segment>
 </net>
@@
 <net name="VIN" class="0">
 <segment>
-<pinref part="J1" gate="G$1" pin="4"/>
 <pinref part="SUPPLY8" gate="G$1" pin="VIN"/>
 <wire x1="30.48" y1="-93.98" x2="30.48" y2="-85.09" width="0.1524" layer="91"/>
-<pinref part="J1" gate="G$1" pin="5"/>
 <wire x1="33.02" y1="-93.98" x2="30.48" y2="-93.98" width="0.1524" layer="91"/>
 <junction x="30.48" y="-93.98"/>
+<pinref part="J3" gate="G$1" pin="4"/>
+<pinref part="J3" gate="G$1" pin="5"/>
 </segment>
 <segment>
@@
 </segment>
 </net>
+<net name="STATUS_1" class="0">
+<segment>
+<pinref part="U1" gate="G$1" pin="(SDA/INT1)PD1"/>
+<wire x1="73.66" y1="2.54" x2="76.2" y2="2.54" width="0.1524" layer="91"/>
+<label x="76.2" y="2.54" size="1.778" layer="95" xref="yes"/>
+</segment>
+<segment>
+<wire x1="167.64" y1="58.42" x2="167.64" y2="60.96" width="0.1524" layer="91"/>
+<label x="167.64" y="60.96" size="1.778" layer="95" rot="R90" xref="yes"/>
+<pinref part="R18" gate="G$1" pin="2"/>
+</segment>
+</net>
+<net name="N$12" class="0">
+<segment>
+<wire x1="167.64" y1="48.26" x2="167.64" y2="45.72" width="0.1524" layer="91"/>
+<pinref part="R18" gate="G$1" pin="1"/>
+<pinref part="LED2" gate="G$1" pin="A"/>
+</segment>
+</net>

Commit message: Update Popping Unit PCB for release, send to board house
Parts:
- added U$20: (no value), blinkinlabs:BUTTON_MOMENTARY
Connections:
- net GND: now also U$20.P
- net RESET: now also U$20.S
Other:
- moved on the sheet: C11, C12, C13, C14, C7, IC2, J2, J3, JP1, JP10, JP11, JP12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

Commit message: Update PoppingUnit board to fix bummer mistake (Arduino remuxes TX, so don't use it as an output channel), update firmware to match
Connections:
- net OUT_1: now also U1.(SDA/INT1)PD1; no longer U1.(TXD1/INT3)PD3
- net STATUS_1: now also U1.(TXD1/INT3)PD3; no longer U1.(SDA/INT1)PD1
Changed lines of the file:
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@@
 </segment>
 <segment>
-<pinref part="U1" gate="G$1" pin="(TXD1/INT3)PD3"/>
-<wire x1="73.66" y1="7.62" x2="76.2" y2="7.62" width="0.1524" layer="91"/>
-<label x="76.2" y="7.62" size="1.778" layer="95" xref="yes"/>
+<pinref part="U1" gate="G$1" pin="(SDA/INT1)PD1"/>
+<wire x1="73.66" y1="2.54" x2="76.2" y2="2.54" width="0.1524" layer="91"/>
+<label x="76.2" y="2.54" size="1.778" layer="95" xref="yes"/>
 </segment>
 </net>
@@
 <net name="STATUS_1" class="0">
 <segment>
-<pinref part="U1" gate="G$1" pin="(SDA/INT1)PD1"/>
-<wire x1="73.66" y1="2.54" x2="76.2" y2="2.54" width="0.1524" layer="91"/>
-<label x="76.2" y="2.54" size="1.778" layer="95" xref="yes"/>
-</segment>
-<segment>
 <wire x1="167.64" y1="58.42" x2="167.64" y2="60.96" width="0.1524" layer="91"/>
 <label x="167.64" y="60.96" size="1.778" layer="95" rot="R90" xref="yes"/>
 <pinref part="R18" gate="G$1" pin="2"/>
 </segment>
-</net>
+<segment>
+<pinref part="U1" gate="G$1" pin="(TXD1/INT3)PD3"/>
+<wire x1="73.66" y1="7.62" x2="76.2" y2="7.62" width="0.1524" layer="91"/>
+<label x="76.2" y="7.62" size="1.778" layer="95" xref="yes"/>
+</segment>
+</net>

Commit message: Update schematic with production component values
Parts:
- C11: value .3uF -> DNP
- C13: value .3uF -> 470nF
- C14: value 100nF -> DNP
- R18, R8: value 1k -> 330
Changed lines of the file:
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@@
 <part name="R1" library="adafruit" deviceset="R-US_" device="R0603" value="180 DNP"/>
 <part name="R2" library="adafruit" deviceset="R-US_" device="R0603" value="10k"/>
-<part name="R8" library="adafruit" deviceset="R-US_" device="R0603" value="1k"/>
+<part name="R8" library="adafruit" deviceset="R-US_" device="R0603" value="330"/>
 <part name="GND12" library="supply1" deviceset="GND" device=""/>
 <part name="C7" library="adafruit" deviceset="C-US" device="C0603K" value="100nF"/>
@@
 <part name="GND18" library="supply1" deviceset="GND" device=""/>
 <part name="GND21" library="supply1" deviceset="GND" device=""/>
-<part name="C11" library="adafruit" deviceset="C-US" device="C0603K" value=".3uF"/>
+<part name="C11" library="adafruit" deviceset="C-US" device="C0603K" value="DNP"/>
 <part name="C12" library="adafruit" deviceset="C-US" device="C0603K" value="100nF"/>
-<part name="C13" library="adafruit" deviceset="C-US" device="C0603K" value=".3uF"/>
-<part name="C14" library="adafruit" deviceset="C-US" device="C0603K" value="100nF"/>
+<part name="C13" library="adafruit" deviceset="C-US" device="C0603K" value="470nF"/>
+<part name="C14" library="adafruit" deviceset="C-US" device="C0603K" value="DNP"/>
 <part name="LED1" library="SparkFun" deviceset="LED" device="5MM"/>
 <part name="J2" library="SparkFun" deviceset="POWER_JACK" device="PTH"/>
@@
 <part name="SUPPLY27" library="SparkFun-Aesthetics" deviceset="2.8V" device=""/>
 <part name="J3" library="con-amp" deviceset="555153-1" device=""/>
-<part name="R18" library="adafruit" deviceset="R-US_" device="R0603" value="1k"/>
+<part name="R18" library="adafruit" deviceset="R-US_" device="R0603" value="330"/>
 <part name="GND29" library="supply1" deviceset="GND" device=""/>
 <part name="LED2" library="SparkFun" deviceset="LED" device="5MM"/>
